File: PCBs/And_gate_using_Transister'.brd (EAGLE design)
At the start: 28 x 26.8 mm, 11 parts, among them T1 BC547, T2 BC547

Commit message: update
Parts:
- moved OUTPUT 24.6 mm to (20.3, 28.9), turned to 180 degrees
- moved B 18.1 mm to (12.7, 28.9), turned to 180 degrees
- moved A 16.9 mm to (5.24, 28.9), turned to 180 degrees
- moved GND 9.62 mm to (14.1, 6.64)
- moved 5V 5.79 mm to (6.41, 6.66)
Routing:
- net N$3: track 38.6 -> 0.00 mm
- net N$6: track 6.66 -> 27.3 mm
- net 5V: track 16.3 -> 0.00 mm
- net N$2: track 10.2 -> 0.00 mm
- net N$4: track 7.62 -> 0.00 mm
- net GND: track 21.9 -> 29.3 mm
- net N$1: track 5.70 -> 0.00 mm
Other:
- board size 28 x 26.8 mm -> 29 x 36.5 mm
- board text added: "Pinwheel Robotics"
- board text added: "care@pinwheel.in"
