File: PCBs/SingleTransistor.sch (EAGLE design)
At the start: 4 parts, among them T1 BC547N

Commit message: Update for Dim width is 42 length is 28 for type 2 pcb
Connections:
- net N$2 renamed T1
Changed lines of the file:
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@@
 </segment>
 </net>
-<net name="N$2" class="0">
+<net name="T1" class="0">
 <segment>
 <pinref part="T1" gate="G$1" pin="B"/>
