File: switch.sch (EAGLE design)
At the start: 3 parts

Commit message: updated
Parts:
- U$1: value MICROBIT_PAD -> pin1
Changed lines of the file:
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@@
 <parts>
 <part name="S1" library="SparkFun-Switches" library_urn="urn:adsk.eagle:library:535" deviceset="MOMENTARY-SWITCH-SPST" device="-PTH-6.0MM" package3d_urn="urn:adsk.eagle:package:40163/1"/>
-<part name="U$1" library="microbit" deviceset="MICROBIT_PAD" device=""/>
+<part name="U$1" library="microbit" deviceset="MICROBIT_PAD" device="" value="pin1"/>
 <part name="U$2" library="microbit" deviceset="MICROBIT_PAD" device=""/>
 </parts>
